File: Polygonus-Universal-Base.kicad_sch (KiCad schematic)
At the start: 14 parts, among them J1 Molex_112_643330100, J2 Conn_01x07, J4 Polygonus_Plugs, U1 f042_wideband_module, U14 f042_wideband_module

Commit message: Getting closer
finished off the main connector, added USB, created case
Parts:
- added J3: Conn_01x05_Male, Connector_PinHeader_2.00mm:PinHeader_1x05_P2.00mm_Vertical, symbol Connector:Conn_01x05_Male
- added J5: USB_B, Simon:BMM-USB, symbol hellen-one-common:USB_B
Connections:
- net GND: now also J4.97 (Pin_97), J4.98 (Pin_98), J3.1 (Pin_1), J3.4 (Pin_4), J5.4 (GND), J5.5 (Shield)
- net USB-: now reaches J4.100 (Pin_100)
- net USB-: now also J3.3 (Pin_3), J5.2 (D-)
- net VBUS: now reaches J4.101 (Pin_101)
- net VBUS: now also J3.5 (Pin_5), J5.1 (VBUS)
- net +3V3: now reaches J4.102 (Pin_102)
- net EXT_SPI_CS: now reaches J4.103 (Pin_103)
- net EXT_SPI_SCK: now reaches J4.104 (Pin_104)
- net EXT_SPI_MISO: now reaches J4.105 (Pin_105)
- net EXT_SPI_MOSI: now reaches J4.106 (Pin_106)
- net USB+: now reaches J4.99 (Pin_99)
- net USB+: now also J3.2 (Pin_2), J5.3 (D+)
- no-connect marks 20 -> 10

Commit message: Added vias, did some DRC checks
Parts:
- removed Motronic_88pin1: Motronic_88pin, Simon:88Pin Motronic BMW, symbol simon rusefi:176122-6_Open_Bosch_88pin
Changed lines of the file:
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@@
-    )
-  )
-  (symbol (lib_id "simon rusefi:176122-6_Open_Bosch_88pin") (at 511.1979 36.681 270) (unit 1)
-    (in_bom yes) (on_board yes) (dnp no)
-    (property "Reference" "Motronic_88pin1" (at 525.5489 70.6408 0)
-      (effects (font (size 1.27 1.27)))
-    )
-    (property "Value" "Motronic_88pin" (at 523.2375 70.6408 0)
-      (effects (font (size 1.27 1.27)))
-    )
-    (property "Footprint" "Simon:88Pin Motronic BMW" (at 522.6279 71.606 0)
-      (effects (font (size 1.27 1.27)) hide)
-    )
-    (property "Datasheet" "DOCUMENTATION" (at 522.6279 48.746 0)
-      (effects (font (size 1.27 1.27)) hide)
-    )
-    (pin "1")
-    (pin "10")
-    (pin "11")
-    (pin "12")
-    (pin "13")
-    (pin "14")
-    (pin "15")
-    (pin "16")
-    (pin "17")
-    (pin "18")
-    (pin "19")
-    (pin "2")
-    (pin "20")
-    (pin "21")
-    (pin "22")
-    (pin "23")
-    (pin "24")
-    (pin "25")
-    (pin "26")
-    (pin "27")
-    (pin "28")
-    (pin "29")
-    (pin "3")
-    (pin "30")
-    (pin "31")
-    (pin "32")
-    (pin "33")
-    (pin "34")
-    (pin "35")
-    (pin "36")
-    (pin "37")
-    (pin "38")
-    (pin "39")
-    (pin "4")
-    (pin "40")
-    (pin "41")
-    (pin "42")
-    (pin "43")
-    (pin "44")
-    (pin "45")
-    (pin "46")
-    (pin "47")
-    (pin "48")
-    (pin "49")
-    (pin "5")
-    (pin "50")
-    (pin "51")
-    (pin "52")
-    (pin "53")
-    (pin "54")
-    (pin "55")
-    (pin "56")
-    (pin "57")
-    (pin "58")
-    (pin "59")
-    (pin "6")
-    (pin "60")
-    (pin "61")
-    (pin "62")
-    (pin "63")
-    (pin "64")
-    (pin "65")
-    (pin "66")
-    (pin "67")
-    (pin "68")
-    (pin "69")
-    (pin "7")
-    (pin "70")
-    (pin "71")
-    (pin "72")
-    (pin "73")
-    (pin "74")
-    (pin "75")
-    (pin "76")
-    (pin "77")
-    (pin "78")
-    (pin "79")
-    (pin "8")
-    (pin "80")
-    (pin "81")
-    (pin "82")
-    (pin "83")
-    (pin "84")
-    (pin "85")
-    (pin "86")
-    (pin "87")
-    (pin "88")
-    (pin "9")
-    (pin "29")
-    (pin "30")
-    (pin "31")
-    (pin "32")
-    (pin "33")
-    (pin "34")
-    (pin "35")
-    (pin "36")
-    (pin "37")
-    (pin "38")
-    (pin "39")
-    (pin "40")
-    (pin "41")
-    (pin "42")
-    (pin "43")
-    (pin "44")
-    (pin "45")
-    (pin "46")
-    (pin "47")
-    (pin "48")
-    (pin "49")
-    (pin "50")
-    (pin "51")
-    (pin "52")
-    (pin "53")
-    (pin "54")
-    (pin "55")
-    (pin "56")
-    (pin "57")
-    (pin "58")
-    (pin "59")
-    (pin "60")
-    (pin "61")
-    (pin "62")
-    (pin "63")
-    (pin "64")
-    (pin "65")
-    (pin "66")
-    (pin "67")
-    (pin "68")
-    (pin "69")
-    (pin "70")
-    (pin "71")
-    (pin "72")
-    (pin "73")
-    (pin "74")
-    (pin "75")
-    (pin "76")
-    (pin "77")
-    (pin "78")
-    (pin "79")
-    (pin "80")
-    (pin "81")
-    (pin "82")
-    (pin "83")
-    (pin "84")
-    (pin "85")
-    (pin "86")
-    (pin "87")
-    (pin "88")
-    (instances
-      (project "Polygonus-Universal-Base"
-        (path "/e63e39d7-6ac0-4ffd-8aa3-1841a4541b55"
-          (reference "Motronic_88pin1") (unit 1)
-        )
-      )
     )
   )

Commit message: Changes to discrete VR
Parts:
- renumbered C10 to C1, C11 to C2, J4 to J2, J5 to J4, J2 to J5, R17 to R1, R18 to R2, R13 to R3, R14 to R4, U14 to U2
Connections:
- net IGN12: now also J5.5 (Pin_5)
Other:
- added sheet VR Module (vr_module_poly.kicad_sch)
- moved on the sheet: J5

Commit message: Added a through hole for the VR and passed DRC
Need to review and publish a gerb
Parts:
- added P1: Pad, Simon:PAD-TH, symbol hellen-one-common:Pad
Connections:
- net +5V: now also J5.2 (Pin_2)
- net 5V_SENSOR_1: no longer J5.2 (Pin_2)
- net IGN12: no longer J5.5 (Pin_5)
- net LS12: now also J5.5 (Pin_5), P1.1 (Pin_1)
Changed lines of the file:
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@@
+    (stroke (width 0) (type default))
+  )
+  (wire (pts (xy 369.57 177.8) (xy 378.46 177.8))
     (stroke (width 0) (type default))
   )
@@
     (effects (font (size 1.27 1.27)) (justify right bottom))
   )
-  (label "5V_SENSOR_1" (at 378.46 170.18 180) (fields_autoplaced)
+  (label "+5V" (at 378.46 170.18 180) (fields_autoplaced)
     (effects (font (size 1.27 1.27)) (justify right bottom))
   )
@@
     (effects (font (size 1.27 1.27)) (justify left bottom))
   )
-  (label "IGN12" (at 370.84 196.85 180) (fields_autoplaced)
+  (label "LS12" (at 370.84 196.85 180) (fields_autoplaced)
     (effects (font (size 1.27 1.27)) (justify right bottom))
   )
@@
     (effects (font (size 1.27 1.27)) (justify right bottom))
   )
-  (label "IGN12" (at 378.46 177.8 180) (fields_autoplaced)
-    (effects (font (size 1.27 1.27)) (justify right bottom))
-  )
   (label "AV3" (at 217.17 78.74 270) (fields_autoplaced)
     (effects (font (size 1.27 1.27)) (justify right bottom))
@@
     (effects (font (size 1.27 1.27)) (justify left bottom))
   )
-  (label "5V_SENSOR_1" (at 370.84 209.55 180) (fields_autoplaced)
+  (label "+5V" (at 370.84 209.55 180) (fields_autoplaced)
     (effects (font (size 1.27 1.27)) (justify right bottom))
   )
@@
   )
   (label "12V_MR" (at 307.34 78.74 270) (fields_autoplaced)
+    (effects (font (size 1.27 1.27)) (justify right bottom))
+  )
+  (label "LS12" (at 377.19 177.8 180) (fields_autoplaced)
     (effects (font (size 1.27 1.27)) (justify right bottom))
   )
@@
         )
       )
+    )
+  )
+  (symbol (lib_id "hellen-one-common:Pad") (at 364.49 177.8 0) (mirror y) (unit 1)
+    (in_bom yes) (on_board yes) (dnp no)
+    (property "Reference" "P1" (at 360.68 177.8 0)
+      (effects (font (size 1.27 1.27)))
+    )
+    (property "Value" "Pad" (at 364.49 180.34 0)
+      (effects (font (size 1.27 1.27)) hide)
+    )
+    (property "Footprint" "Simon:PAD-TH" (at 364.49 181.61 0)
+      (effects (font (size 1.27 1.27)) hide)
+    )
+    (property "Datasheet" "~" (at 364.49 177.8 0)
+      (effects (font (size 1.27 1.27)) hide)
+    )
+    (pin "1")
+    (instances
+      (project "Polygonus-Universal-Base"
+        (path "/e63e39d7-6ac0-4ffd-8aa3-1841a4541b55"
+          (reference "P1") (unit 1)
+        )
+      )

Commit message: fixed plug pin numbering error
Parts:
- J1: footprint Simon:Molex_112_643330100 -> Miata NC 120 pin
Changed lines of the file:
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@@
       (effects (font (size 1.27 1.27)))
     )
-    (property "Footprint" "Simon:Molex_112_643330100" (at 31.75 64.77 0)
+    (property "Footprint" "Miata NC 120 pin" (at 31.75 64.77 0)
       (effects (font (size 1.27 1.27)) hide)
     )

Commit message: fixed issues: 10, 6, 5, 4 and 2
Parts:
- added P2, P3, P4, P5, P6: Pad, Simon:PAD-TH, symbol hellen-one-common:Pad
- J1: footprint Miata NC 120 pin -> Simon:Molex_112_643330100
Connections:
- net 12V_MR: now also P1.1 (Pin_1), P6.1 (Pin_1)
- net 5V_SENSOR_1: no longer J1.15
- net 5V_SENSOR_2: no longer J1.11
- net CAN2+: now also J1.15
- net CAN2-: now also J1.11
- net ExtraLSA: now also P2.1 (Pin_1)
- net ExtraLSB: now also P3.1 (Pin_1)
- net LS12: no longer J5.5 (Pin_5), P1.1 (Pin_1)
- net LS12ADD: now also P5.1 (Pin_1)
- net LS9ADD: now also P4.1 (Pin_1)
- net VR2+: now also J2.78 (Pin_78)
- no-connect marks 10 -> 9
Other:
- moved on the sheet: P1

Commit message: V1.0 published
Connections:
- net HS1: now also J1.28, J2.65 (Pin_65); no longer J1.26, J2.68 (Pin_68)
- net HS2: now also J1.27, J2.66 (Pin_66); no longer J1.25, J2.67 (Pin_67)
- net HS3: now also J1.25, J2.67 (Pin_67); no longer J1.27, J2.66 (Pin_66)
- net HS4: now also J1.26, J2.68 (Pin_68); no longer J1.28, J2.65 (Pin_65)
- net LS12: now also J5.5 (Pin_5)
Changed lines of the file:
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@@
-		)
-	)
-	(label "HS3"
-		(at 313.69 111.76 180)
-		(fields_autoplaced yes)
-		(effects
-			(font
-				(size 1.27 1.27)
-			)
-			(justify right bottom)
 		)
 	)
@@
 		)
 	)
+	(label "HS3"
+		(at 313.69 114.3 180)
+		(fields_autoplaced yes)
+		(effects
+			(font
+				(size 1.27 1.27)
+			)
+			(justify right bottom)
+		)
+	)
 	(label "AV11"
 		(at 378.46 175.26 180)
@@
 		)
 	)
+	(label "HS1"
+		(at 105.41 78.74 270)
+		(fields_autoplaced yes)
+		(effects
+			(font
+				(size 1.27 1.27)
+			)
+			(justify right bottom)
+		)
+	)
 	(label "LS16"
 		(at 224.79 186.69 180)
@@
 		)
 	)
+	(label "HS2"
+		(at 102.87 78.74 270)
+		(fields_autoplaced yes)
+		(effects
+			(font
+				(size 1.27 1.27)
+			)
+			(justify right bottom)
+		)
+	)
 	(label "CAN_TX2"
 		(at 160.02 261.5873 180)
@@
 		)
 	)
-	(label "HS1"
-		(at 313.69 116.84 180)
-		(fields_autoplaced yes)
-		(effects
-			(font
-				(size 1.27 1.27)
-			)
-			(justify right bottom)
-		)
-	)
 	(label "AV6"
 		(at 262.89 171.45 180)
@@
 		)
 	)
+	(label "HS4"
+		(at 100.33 78.74 270)
+		(fields_autoplaced yes)
+		(effects
+			(font
+				(size 1.27 1.27)
+			)
+			(justify right bottom)
+		)
+	)
 	(label "CAN2+"
 		(at 313.69 129.54 180)
@@
 		)
 	)
+	(label "HS2"
+		(at 313.69 111.76 180)
+		(fields_autoplaced yes)
+		(effects
+			(font
+				(size 1.27 1.27)
+			)
+			(justify right bottom)
+		)
+	)
 	(label "IGN5"
 		(at 146.05 78.74 270)
@@
 		)
 	)
-	(label "HS2"
-		(at 97.79 78.74 270)
-		(fields_autoplaced yes)
-		(effects
-			(font
-				(size 1.27 1.27)
-			)
-			(justify right bottom)
-		)
-	)
 	(label "12V_PROT"
 		(at 262.89 113.03 180)
@@
 		)
 	)
+	(label "HS3"
+		(at 97.79 78.74 270)
+		(fields_autoplaced yes)
+		(effects
+			(font
+				(size 1.27 1.27)
+			)
+			(justify right bottom)
+		)
+	)
 	(label "IGN5"
 		(at 224.79 156.21 180)
@@
 		)
 	)
-	(label "HS4"
-		(at 313.69 109.22 180)
-		(fields_autoplaced yes)
-		(effects
-			(font
-				(size 1.27 1.27)
-			)
-			(justify right bottom)
-		)
-	)
 	(label "USB+"
 		(at 288.29 115.57 180)
@@
 		)
 	)
-	(label "HS3"
-		(at 102.87 78.74 270)
-		(fields_autoplaced yes)
-		(effects
-			(font
-				(size 1.27 1.27)
-			)
-			(justify right bottom)
-		)
-	)
 	(label "LS9ADD"
 		(at 80.01 171.45 0)
@@
 		)
 	)
-	(label "HS1"
-		(at 100.33 78.74 270)
-		(fields_autoplaced yes)
-		(effects
-			(font
-				(size 1.27 1.27)
-			)
-			(justify right bottom)
-		)
-	)
 	(label "STEPB2"
 		(at 168.91 78.74 270)
@@
 	)
 	(label "HS4"
-		(at 105.41 78.74 270)
+		(at 313.69 116.84 180)
 		(fields_autoplaced yes)
 		(effects
@@
 		)
 	)
+	(label "HS1"
+		(at 313.69 109.22 180)
+		(fields_autoplaced yes)
+		(effects
+			(font
+				(size 1.27 1.27)
+			)
+			(justify right bottom)
+		)
+	)
 	(label "IGN7"
 		(at 231.14 259.08 180)
@@
 		)
 	)
-	(label "HS2"
-		(at 313.69 114.3 180)
-		(fields_autoplaced yes)
-		(effects
-			(font
-				(size 1.27 1.27)
-			)
-			(justify right bottom)
-		)
-	)
 	(label "LS8"
 		(at 266.7 78.74 270)
@@
 	)
 	(label "LS12"
-		(at 377.19 177.8 180)
-		(fields_autoplaced yes)
-		(effects
+		(at 378.46 177.8 180)
+		(fields_autoplaced yes)
+		(effects

Commit message: Fixed trigger scope
Connections:
- net AV11: no longer J5.4 (Pin_4)
- net VR2+: no longer J2.78 (Pin_78)
- new net Scope: J2.78 (Pin_78), J5.4 (Pin_4)
