File: VR conditioner.kicad_sch (KiCad schematic)
At the start: 15 parts, among them U3 MAX9924

Commit message: Changes to discrete VR
Parts:
- renumbered C4 to C23, C5 to C24, C6 to C25, JP2 to JP1, R2 to R25, R3 to R26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
