File: etb-9201.kicad_sch (KiCad schematic)
At the start: 5 parts, among them U2 TLE9201SG

Commit message: Changes to discrete VR
Parts:
- renumbered C1 to C3, C2 to C4, C3 to C5, R1 to R5, U2 to U3
Changed lines of the file:
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@@
   (symbol (lib_id "Device:R") (at 68.58 57.15 270) (unit 1)
     (in_bom yes) (on_board yes) (dnp no)
-    (property "Reference" "R1" (at 68.58 59.69 90)
+    (property "Reference" "R5" (at 68.58 59.69 90)
       (effects (font (size 1.27 1.27)))
     )
@@
       (project "Polygonus-Universal-Base"
         (path "/e63e39d7-6ac0-4ffd-8aa3-1841a4541b55/eb1c8308-a44a-4a4b-a646-1cfc69b467a3"
-          (reference "R1") (unit 1)
-        )
-        (path "/e63e39d7-6ac0-4ffd-8aa3-1841a4541b55/8bc5218e-e3ef-4de7-bea4-c8f4c6a87c8a"
-          (reference "R12") (unit 1)
+          (reference "R5") (unit 1)
+        )
+        (path "/e63e39d7-6ac0-4ffd-8aa3-1841a4541b55/8bc5218e-e3ef-4de7-bea4-c8f4c6a87c8a"
+          (reference "R35") (unit 1)
         )
       )
@@
         )
         (path "/e63e39d7-6ac0-4ffd-8aa3-1841a4541b55/eb1c8308-a44a-4a4b-a646-1cfc69b467a3"
-          (reference "#PWR031") (unit 1)
-        )
-        (path "/e63e39d7-6ac0-4ffd-8aa3-1841a4541b55/8bc5218e-e3ef-4de7-bea4-c8f4c6a87c8a"
-          (reference "#PWR049") (unit 1)
+          (reference "#PWR052") (unit 1)
+        )
+        (path "/e63e39d7-6ac0-4ffd-8aa3-1841a4541b55/8bc5218e-e3ef-4de7-bea4-c8f4c6a87c8a"
+          (reference "#PWR0131") (unit 1)
         )
       )
@@
         )
         (path "/e63e39d7-6ac0-4ffd-8aa3-1841a4541b55/eb1c8308-a44a-4a4b-a646-1cfc69b467a3"
-          (reference "#PWR027") (unit 1)
-        )
-        (path "/e63e39d7-6ac0-4ffd-8aa3-1841a4541b55/8bc5218e-e3ef-4de7-bea4-c8f4c6a87c8a"
-          (reference "#PWR028") (unit 1)
+          (reference "#PWR048") (unit 1)
+        )
+        (path "/e63e39d7-6ac0-4ffd-8aa3-1841a4541b55/8bc5218e-e3ef-4de7-bea4-c8f4c6a87c8a"
+          (reference "#PWR0127") (unit 1)
         )
       )
@@
         )
         (path "/e63e39d7-6ac0-4ffd-8aa3-1841a4541b55/eb1c8308-a44a-4a4b-a646-1cfc69b467a3"
-          (reference "#PWR052") (unit 1)
-        )
-        (path "/e63e39d7-6ac0-4ffd-8aa3-1841a4541b55/8bc5218e-e3ef-4de7-bea4-c8f4c6a87c8a"
-          (reference "#PWR053") (unit 1)
+          (reference "#PWR047") (unit 1)
+        )
+        (path "/e63e39d7-6ac0-4ffd-8aa3-1841a4541b55/8bc5218e-e3ef-4de7-bea4-c8f4c6a87c8a"
+          (reference "#PWR0126") (unit 1)
         )
       )
@@
         )
         (path "/e63e39d7-6ac0-4ffd-8aa3-1841a4541b55/eb1c8308-a44a-4a4b-a646-1cfc69b467a3"
-          (reference "#PWR029") (unit 1)
-        )
-        (path "/e63e39d7-6ac0-4ffd-8aa3-1841a4541b55/8bc5218e-e3ef-4de7-bea4-c8f4c6a87c8a"
-          (reference "#PWR030") (unit 1)
+          (reference "#PWR049") (unit 1)
+        )
+        (path "/e63e39d7-6ac0-4ffd-8aa3-1841a4541b55/8bc5218e-e3ef-4de7-bea4-c8f4c6a87c8a"
+          (reference "#PWR0128") (unit 1)
         )
       )
@@
         )
         (path "/e63e39d7-6ac0-4ffd-8aa3-1841a4541b55/eb1c8308-a44a-4a4b-a646-1cfc69b467a3"
-          (reference "#PWR050") (unit 1)
-        )
-        (path "/e63e39d7-6ac0-4ffd-8aa3-1841a4541b55/8bc5218e-e3ef-4de7-bea4-c8f4c6a87c8a"
           (reference "#PWR051") (unit 1)
         )
+        (path "/e63e39d7-6ac0-4ffd-8aa3-1841a4541b55/8bc5218e-e3ef-4de7-bea4-c8f4c6a87c8a"
+          (reference "#PWR0130") (unit 1)
+        )
       )
     )
@@
   (symbol (lib_id "Simon:TLE9201SG") (at 97.79 63.5 0) (unit 1)
     (in_bom yes) (on_board yes) (dnp no) (fields_autoplaced)
-    (property "Reference" "U2" (at 97.155 46.99 0)
+    (property "Reference" "U3" (at 97.155 46.99 0)
       (effects (font (size 1.27 1.27)))
     )
@@
       (project "Polygonus-Universal-Base"
         (path "/e63e39d7-6ac0-4ffd-8aa3-1841a4541b55/eb1c8308-a44a-4a4b-a646-1cfc69b467a3"
-          (reference "U2") (unit 1)
-        )
-        (path "/e63e39d7-6ac0-4ffd-8aa3-1841a4541b55/8bc5218e-e3ef-4de7-bea4-c8f4c6a87c8a"
-          (reference "U8") (unit 1)
+          (reference "U3") (unit 1)
+        )
+        (path "/e63e39d7-6ac0-4ffd-8aa3-1841a4541b55/8bc5218e-e3ef-4de7-bea4-c8f4c6a87c8a"
+          (reference "U15") (unit 1)
         )
       )
@@
   (symbol (lib_id "power:+3.3V") (at 109.22 74.93 270) (unit 1)
     (in_bom yes) (on_board yes) (dnp no) (fields_autoplaced)
-    (property "Reference" "#PWR0128" (at 105.41 74.93 0)
+    (property "Reference" "#PWR0129" (at 105.41 74.93 0)
       (effects (font (size 1.27 1.27)) hide)
     )
@@
       (project "Polygonus-Universal-Base"
         (path "/e63e39d7-6ac0-4ffd-8aa3-1841a4541b55/8bc5218e-e3ef-4de7-bea4-c8f4c6a87c8a"
-          (reference "#PWR0128") (unit 1)
-        )
-        (path "/e63e39d7-6ac0-4ffd-8aa3-1841a4541b55/eb1c8308-a44a-4a4b-a646-1cfc69b467a3"
-          (reference "#PWR0115") (unit 1)
+          (reference "#PWR0129") (unit 1)
+        )
+        (path "/e63e39d7-6ac0-4ffd-8aa3-1841a4541b55/eb1c8308-a44a-4a4b-a646-1cfc69b467a3"
+          (reference "#PWR050") (unit 1)
         )
       )
@@
   (symbol (lib_id "Device:C_Small") (at 114.3 60.325 0) (unit 1)
     (in_bom yes) (on_board yes) (dnp no)
-    (property "Reference" "C3" (at 116.6368 59.1566 0)
+    (property "Reference" "C5" (at 116.6368 59.1566 0)
       (effects (font (size 1.27 1.27)) (justify left))
     )
@@
       (project "Polygonus-Universal-Base"
         (path "/e63e39d7-6ac0-4ffd-8aa3-1841a4541b55/eb1c8308-a44a-4a4b-a646-1cfc69b467a3"
-          (reference "C3") (unit 1)
-        )
-        (path "/e63e39d7-6ac0-4ffd-8aa3-1841a4541b55/8bc5218e-e3ef-4de7-bea4-c8f4c6a87c8a"
-          (reference "C9") (unit 1)
+          (reference "C5") (unit 1)
+        )
+        (path "/e63e39d7-6ac0-4ffd-8aa3-1841a4541b55/8bc5218e-e3ef-4de7-bea4-c8f4c6a87c8a"
+          (reference "C28") (unit 1)
         )
       )
@@
   (symbol (lib_id "Device:C") (at 80.645 46.99 0) (unit 1)
     (in_bom yes) (on_board yes) (dnp no)
-    (property "Reference" "C1" (at 83.566 45.8216 0)
+    (property "Reference" "C3" (at 83.566 45.8216 0)
       (effects (font (size 1.27 1.27)) (justify left))
     )
@@
       (project "Polygonus-Universal-Base"
         (path "/e63e39d7-6ac0-4ffd-8aa3-1841a4541b55/eb1c8308-a44a-4a4b-a646-1cfc69b467a3"
-          (reference "C1") (unit 1)
-        )
-        (path "/e63e39d7-6ac0-4ffd-8aa3-1841a4541b55/8bc5218e-e3ef-4de7-bea4-c8f4c6a87c8a"
-          (reference "C7") (unit 1)
+          (reference "C3") (unit 1)
+        )
+        (path "/e63e39d7-6ac0-4ffd-8aa3-1841a4541b55/8bc5218e-e3ef-4de7-bea4-c8f4c6a87c8a"
+          (reference "C26") (unit 1)
         )
       )
@@
   (symbol (lib_id "power:+3.3V") (at 64.77 57.15 90) (unit 1)
     (in_bom yes) (on_board yes) (dnp no) (fields_autoplaced)
-    (property "Reference" "#PWR062" (at 68.58 57.15 0)
+    (property "Reference" "#PWR0125" (at 68.58 57.15 0)
       (effects (font (size 1.27 1.27)) hide)
     )
@@
       (project "Polygonus-Universal-Base"
         (path "/e63e39d7-6ac0-4ffd-8aa3-1841a4541b55/8bc5218e-e3ef-4de7-bea4-c8f4c6a87c8a"
-          (reference "#PWR062") (unit 1)
-        )
-        (path "/e63e39d7-6ac0-4ffd-8aa3-1841a4541b55/eb1c8308-a44a-4a4b-a646-1cfc69b467a3"
-          (reference "#PWR040") (unit 1)
+          (reference "#PWR0125") (unit 1)
+        )
+        (path "/e63e39d7-6ac0-4ffd-8aa3-1841a4541b55/eb1c8308-a44a-4a4b-a646-1cfc69b467a3"
+          (reference "#PWR046") (unit 1)
         )
       )
@@
   (symbol (lib_id "Device:C_Small") (at 114.3 48.895 0) (unit 1)
     (in_bom yes) (on_board yes) (dnp no)
-    (property "Reference" "C2" (at 116.6368 47.7266 0)
+    (property "Reference" "C4" (at 116.6368 47.7266 0)
       (effects (font (size 1.27 1.27)) (justify left))
     )
@@
       (project "Polygonus-Universal-Base"
         (path "/e63e39d7-6ac0-4ffd-8aa3-1841a4541b55/eb1c8308-a44a-4a4b-a646-1cfc69b467a3"
-          (reference "C2") (unit 1)
-        )
-        (path "/e63e39d7-6ac0-4ffd-8aa3-1841a4541b55/8bc5218e-e3ef-4de7-bea4-c8f4c6a87c8a"
-          (reference "C8") (unit 1)
-        )
-      )
+          (reference "C4") (unit 1)
+        )
+        (path "/e63e39d7-6ac0-4ffd-8aa3-1841a4541b55/8bc5218e-e3ef-4de7-bea4-c8f4c6a87c8a"
+          (reference "C27") (unit 1)
+        )
+      )

Commit message: V1.0 published
Parts:
- renumbered C3 to C26, C4 to C27, C5 to C28, R5 to R35, U3 to U15
Changed lines of the file:
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@@
 		(on_board yes)
 		(dnp no)
-		(property "Reference" "R5"
+		(property "Reference" "R35"
 			(at 68.58 59.69 90)
 			(effects
@@
 		(dnp no)
 		(fields_autoplaced yes)
-		(property "Reference" "#PWR052"
+		(property "Reference" "#PWR0131"
 			(at 114.3 69.215 0)
 			(effects
@@
 		(dnp no)
 		(fields_autoplaced yes)
-		(property "Reference" "#PWR048"
+		(property "Reference" "#PWR0127"
 			(at 78.74 72.39 0)
 			(effects
@@
 		(dnp no)
 		(fields_autoplaced yes)
-		(property "Reference" "#PWR047"
+		(property "Reference" "#PWR0126"
 			(at 80.645 36.83 0)
 			(effects
@@
 		(dnp no)
 		(fields_autoplaced yes)
-		(property "Reference" "#PWR049"
+		(property "Reference" "#PWR0128"
 			(at 78.74 74.93 0)
 			(effects
@@
 		(dnp no)
 		(fields_autoplaced yes)
-		(property "Reference" "#PWR051"
+		(property "Reference" "#PWR0130"
 			(at 114.3 40.005 0)
 			(effects
@@
 		(dnp no)
 		(fields_autoplaced yes)
-		(property "Reference" "U3"
+		(property "Reference" "U15"
 			(at 97.155 46.99 0)
 			(effects
@@
 		(on_board yes)
 		(dnp no)
-		(property "Reference" "C5"
+		(property "Reference" "C28"
 			(at 116.6368 59.1566 0)
 			(effects
@@
 		(on_board yes)
 		(dnp no)
-		(property "Reference" "C3"
+		(property "Reference" "C26"
 			(at 83.566 45.8216 0)
 			(effects
@@
 		(on_board yes)
 		(dnp no)
-		(property "Reference" "C4"
+		(property "Reference" "C27"
 			(at 116.6368 47.7266 0)
 			(effects

Commit message: Fixed trigger scope
Parts:
- renumbered C26 to C3, C27 to C4, C28 to C5, R35 to R5, U15 to U3
Changed lines of the file:
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@@
 (kicad_sch
-	(version 20231120)
+	(version 20250114)
 	(generator "eeschema")
-	(generator_version "8.0")
+	(generator_version "9.0")
 	(paper "A4")
 	(title_block
@@
 		(company "FutureProofPerformance.com")
 	)
+	(text "IFX9201 also acceptable"
+		(exclude_from_sim no)
+		(at 86.36 80.01 0)
+		(effects
+			(font
+				(size 1.27 1.27)
+			)
+			(justify left bottom)
+		)
+	)
 	(junction
 		(at 80.645 53.34)
@@
 		)
 	)
-	(text "IFX9201 also acceptable"
-		(exclude_from_sim no)
-		(at 86.36 80.01 0)
+	(hierarchical_label "OUT+"
+		(shape output)
+		(at 118.745 53.34 0)
 		(effects
 			(font
 				(size 1.27 1.27)
 			)
-			(justify left bottom)
-		)
-	)
-	(hierarchical_label "OUT+"
-		(shape output)
-		(at 118.745 53.34 0)
-		(fields_autoplaced yes)
+			(justify left)
+		)
+	)
+	(hierarchical_label "PWM"
+		(shape input)
+		(at 78.105 66.04 180)
 		(effects
 			(font
 				(size 1.27 1.27)
 			)
-			(justify left)
-		)
-	)
-	(hierarchical_label "PWM"
+			(justify right)
+		)
+	)
+	(hierarchical_label "DIR"
 		(shape input)
-		(at 78.105 66.04 180)
-		(fields_autoplaced yes)
+		(at 78.105 63.5 180)
 		(effects
 			(font
@@
 		)
 	)
-	(hierarchical_label "DIR"
+	(hierarchical_label "12V_SUPPLY"
 		(shape input)
-		(at 78.105 63.5 180)
-		(fields_autoplaced yes)
+		(at 54.61 48.26 180)
 		(effects
 			(font
@@
 		)
 	)
-	(hierarchical_label "12V_SUPPLY"
+	(hierarchical_label "DIS"
 		(shape input)
-		(at 54.61 48.26 180)
-		(fields_autoplaced yes)
+		(at 77.47 60.96 180)
 		(effects
 			(font
@@
 		)
 	)
-	(hierarchical_label "DIS"
-		(shape input)
-		(at 77.47 60.96 180)
-		(fields_autoplaced yes)
-		(effects
-			(font
-				(size 1.27 1.27)
-			)
-			(justify right)
-		)
-	)
 	(hierarchical_label "OUT-"
 		(shape output)
 		(at 118.745 55.88 0)
-		(fields_autoplaced yes)
 		(effects
 			(font
@@
 		(on_board yes)
 		(dnp no)
-		(property "Reference" "R35"
+		(property "Reference" "R5"
 			(at 68.58 59.69 90)
 			(effects
@@
 		(dnp no)
 		(fields_autoplaced yes)
-		(property "Reference" "#PWR0131"
+		(property "Reference" "#PWR052"
 			(at 114.3 69.215 0)
 			(effects
@@
 		(dnp no)
 		(fields_autoplaced yes)
-		(property "Reference" "#PWR0127"
+		(property "Reference" "#PWR048"
 			(at 78.74 72.39 0)
 			(effects
@@
 		(dnp no)
 		(fields_autoplaced yes)
-		(property "Reference" "#PWR0126"
+		(property "Reference" "#PWR047"
 			(at 80.645 36.83 0)
 			(effects
@@
 		(dnp no)
 		(fields_autoplaced yes)
-		(property "Reference" "#PWR0128"
+		(property "Reference" "#PWR049"
 			(at 78.74 74.93 0)
 			(effects
@@
 		(dnp no)
 		(fields_autoplaced yes)
-		(property "Reference" "#PWR0130"
+		(property "Reference" "#PWR051"
 			(at 114.3 40.005 0)
 			(effects
@@
 		(dnp no)
 		(fields_autoplaced yes)
-		(property "Reference" "U15"
+		(property "Reference" "U3"
 			(at 97.155 46.99 0)
 			(effects
@@
 		(dnp no)
 		(fields_autoplaced yes)
-		(property "Reference" "#PWR0129"
+		(property "Reference" "#PWR050"
 			(at 105.41 74.93 0)
 			(effects
@@
 		(on_board yes)
 		(dnp no)
-		(property "Reference" "C28"
+		(property "Reference" "C5"
 			(at 116.6368 59.1566 0)
 			(effects
@@
 		(on_board yes)
 		(dnp no)
-		(property "Reference" "C26"
+		(property "Reference" "C3"
 			(at 83.566 45.8216 0)
 			(effects
@@
 		(dnp no)
 		(fields_autoplaced yes)
-		(property "Reference" "#PWR0125"
+		(property "Reference" "#PWR046"
 			(at 68.58 57.15 0)
 			(effects
@@
 		(on_board yes)
 		(dnp no)
-		(property "Reference" "C27"
+		(property "Reference" "C4"
 			(at 116.6368 47.7266 0)
 			(effects
