File: vr_module_poly.kicad_sch (KiCad schematic)
At the start: 43 parts, among them U1 MAX9142, U2 NC7SB3157P6X, U3 74HC02, U4 NC7SB3157P6X, U5 SRV05-4, U6 MCP6004

Commit message: Fixed trigger scope
Parts:
- renumbered C9 to C10, C1 to C11, C2 to C12, C12 to C13, C4 to C14, C14 to C15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
